File: shema/shema.sch (EAGLE design)
At the start: 11 parts, among them IC2 TINY13V-10SSU, T1 2N2222

Commit message: #
Parts:
- D1, D2, D3: device SparkFun-LED:LED3MM -> SparkFun-LED:LED-3MM-NO_SILK
- T1: value 2N2222 -> 2SC945; device adafruit:2N2222 -> transistor:2SC945
- renumbered PAD1 to -, PAD2 to +
Other:
- moved on the sheet: C1
Changed lines of the file:
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@@
 <part name="S1" library="SparkFun-Switches" deviceset="MOMENTARY-SWITCH-SPST" device="-SMD-4.5MM" value="S1"/>
 <part name="R1" library="SparkFun-Resistors" deviceset="2MOHMS" device="-0603-1/10W-1%" value="1K"/>
-<part name="PAD1" library="wirepad" deviceset="2,54/0,8" device=""/>
-<part name="PAD2" library="wirepad" deviceset="2,54/0,8" device=""/>
-<part name="T1" library="adafruit" deviceset="2N2222" device=""/>
+<part name="-" library="wirepad" deviceset="2,54/0,8" device=""/>
+<part name="+" library="wirepad" deviceset="2,54/0,8" device=""/>
+<part name="T1" library="transistor" deviceset="2SC945" device=""/>
 <part name="GND2" library="supply1" deviceset="GND" device=""/>
 <part name="R2" library="SparkFun-Resistors" deviceset="2MOHMS" device="-0603-1/10W-1%" value="10K"/>
@@
 <part name="GND4" library="supply1" deviceset="GND" device=""/>
 <part name="P+3" library="supply1" deviceset="+5V" device=""/>
-<part name="D1" library="SparkFun-LED" deviceset="LED" device="3MM"/>
-<part name="D2" library="SparkFun-LED" deviceset="LED" device="3MM"/>
-<part name="D3" library="SparkFun-LED" deviceset="LED" device="3MM"/>
+<part name="D1" library="SparkFun-LED" deviceset="LED" device="-3MM-NO_SILK"/>
+<part name="D2" library="SparkFun-LED" deviceset="LED" device="-3MM-NO_SILK"/>
+<part name="D3" library="SparkFun-LED" deviceset="LED" device="-3MM-NO_SILK"/>
 <part name="P+4" library="supply1" deviceset="+5V" device=""/>
 <part name="C1" library="SparkFun-Capacitors" deviceset="560PF" device="-0603-50V-5%" value="1000pF"/>
@@
 <instance part="S1" gate="G$1" x="43.18" y="58.42" rot="R90"/>
 <instance part="R1" gate="G$1" x="45.72" y="86.36" rot="R180"/>
-<instance part="PAD1" gate="P" x="83.82" y="50.8" rot="R270"/>
-<instance part="PAD2" gate="P" x="93.98" y="50.8" rot="R270"/>
-<instance part="T1" gate="G$1" x="25.4" y="73.66" rot="MR0"/>
-<instance part="GND2" gate="1" x="22.86" y="58.42"/>
+<instance part="-" gate="P" x="83.82" y="50.8" rot="R270"/>
+<instance part="+" gate="P" x="93.98" y="50.8" rot="R270"/>
+<instance part="T1" gate="G$1" x="25.4" y="73.66" smashed="yes" rot="MR0">
+<attribute name="NAME" x="35.56" y="81.28" size="1.778" layer="95" rot="MR0"/>
+<attribute name="VALUE" x="35.56" y="78.74" size="1.778" layer="96" rot="MR0"/>
+</instance>
+<instance part="GND2" gate="1" x="17.78" y="58.42"/>
 <instance part="R2" gate="G$1" x="53.34" y="58.42" rot="R270"/>
 <instance part="GND3" gate="1" x="43.18" y="48.26"/>
@@
 <attribute name="VALUE" x="20.32" y="104.14" size="1.778" layer="96" rot="R90"/>
 </instance>
-<instance part="C1" gate="G$1" x="30.48" y="58.42"/>
+<instance part="C1" gate="G$1" x="25.4" y="58.42"/>
 </instances>
 <busses>
@@
 <nets>
 <net name="GND" class="0">
-<segment>
-<pinref part="GND2" gate="1" pin="GND"/>
-<pinref part="T1" gate="G$1" pin="E"/>
-<wire x1="22.86" y1="60.96" x2="22.86" y2="68.58" width="0.1524" layer="91"/>
-</segment>
 <segment>
 <pinref part="IC2" gate="G$1" pin="GND"/>
@@
 <wire x1="43.18" y1="53.34" x2="43.18" y2="50.8" width="0.1524" layer="91"/>
 <pinref part="C1" gate="G$1" pin="2"/>
-<wire x1="30.48" y1="55.88" x2="30.48" y2="50.8" width="0.1524" layer="91"/>
-<wire x1="30.48" y1="50.8" x2="43.18" y2="50.8" width="0.1524" layer="91"/>
+<wire x1="25.4" y1="55.88" x2="25.4" y2="50.8" width="0.1524" layer="91"/>
+<wire x1="25.4" y1="50.8" x2="43.18" y2="50.8" width="0.1524" layer="91"/>
 </segment>
 <segment>
-<pinref part="PAD1" gate="P" pin="P"/>
+<pinref part="-" gate="P" pin="P"/>
 <pinref part="GND4" gate="1" pin="GND"/>
 <wire x1="83.82" y1="48.26" x2="83.82" y2="40.64" width="0.1524" layer="91"/>
+<junction x="83.82" y="48.26"/>
+<junction x="83.82" y="40.64"/>
+</segment>
+<segment>
+<pinref part="GND2" gate="1" pin="GND"/>
+<wire x1="17.78" y1="60.96" x2="17.78" y2="68.58" width="0.1524" layer="91"/>
+<pinref part="T1" gate="G$1" pin="E"/>
+<wire x1="17.78" y1="68.58" x2="22.86" y2="68.58" width="0.1524" layer="91"/>
 </segment>
 </net>
@@
 </segment>
 <segment>
-<pinref part="PAD2" gate="P" pin="P"/>
+<pinref part="+" gate="P" pin="P"/>
 <pinref part="P+3" gate="1" pin="+5V"/>
 <wire x1="93.98" y1="48.26" x2="93.98" y2="40.64" width="0.1524" layer="91"/>
+<junction x="93.98" y="40.64"/>
+<junction x="93.98" y="48.26"/>
 </segment>
 <segment>
@@
 <junction x="53.34" y="78.74"/>
 <pinref part="C1" gate="G$1" pin="1"/>
-<wire x1="30.48" y1="63.5" x2="30.48" y2="68.58" width="0.1524" layer="91"/>
-<wire x1="30.48" y1="68.58" x2="43.18" y2="68.58" width="0.1524" layer="91"/>
+<wire x1="25.4" y1="63.5" x2="25.4" y2="68.58" width="0.1524" layer="91"/>
+<wire x1="25.4" y1="68.58" x2="43.18" y2="68.58" width="0.1524" layer="91"/>
 <junction x="43.18" y="68.58"/>
 </segment>
