File: shema/shema.brd (EAGLE design)
At the start: 26 x 29 mm, 11 parts, among them IC2 TINY13V-10SSU, T1 2SC945

Commit message: %
Parts:
- moved R1 17.5 mm to (18.7, 4.10), turned to 180 degrees
- moved C1 9.01 mm to (17.1, 9.14)
- moved IC2 8.06 mm to (22.8, 18.2)
- moved T1 3.64 mm to (12.3, 6.44), turned to 270 degrees
- moved R2 3.54 mm to (22.5, 7.90)
- moved S1 1.25 mm to (14.0, 14.8), turned to 0 degrees
- moved D2 1.00 mm to (5.05, 14.7)
Routing:
- net +5V: track 0.00 -> 91.3 mm
- net N$6: track 0.00 -> 48.3 mm
- net GND: track 0.00 -> 38.4 mm
- net N$2: track 0.00 -> 28.4 mm
- net N$1: track 0.00 -> 12.0 mm
- net N$3: track 0.00 -> 5.69 mm

Commit message: ~
Parts:
- moved C1 14.3 mm to (12.4, 22.6), turned to 180 degrees
- moved R1 6.58 mm to (19.7, 10.6)
- moved R2 5.10 mm to (23.5, 12.9)
- moved IC2 1.41 mm to (21.8, 19.2)
Routing:
- net +5V: track 91.3 -> 37.3 mm
- net N$2: track 28.4 -> 21.0 mm
- net N$6: track 48.3 -> 41.4 mm
- net N$1: track 12.0 -> 6.21 mm
- net GND: track 38.4 -> 33.5 mm
- net N$3: track 5.69 -> 9.65 mm
